Commit message: fixed some urdf bugs

File: Model/panda_arm.urdf (robot description, URDF)
Before this commit: robot panda, 8 links, 7 joints
Links:
- link link0: geometry visual mesh filename=../../Model/meshes/visual/link0.obj
- link link1: geometry visual mesh filename=../../Model/meshes/visual/link1.obj
- link link2: geometry visual mesh filename=../../Model/meshes/visual/link2.obj
- link link3: geometry visual mesh filename=../../Model/meshes/visual/link3.obj
- link link4: geometry visual mesh filename=../../Model/meshes/visual/link4.obj
- link link5: geometry visual mesh filename=../../Model/meshes/visual/link5.obj
- link link6: geometry visual mesh filename=../../Model/meshes/visual/link6.obj
- link link7: geometry visual mesh filename=../../Model/meshes/visual/link7.obj

File: Model/panda_arm_hand.urdf (robot description, URDF)
Before this commit: robot panda_hand, 10 links, 9 joints
Links:
- link leftfinger: geometry visual mesh filename=../../Model/meshes/visual/finger.obj
- link link0: geometry visual mesh filename=../../Model/meshes/visual/link0.obj
- link link1: geometry visual mesh filename=../../Model/meshes/visual/link1.obj
- link link2: geometry visual mesh filename=../../Model/meshes/visual/link2.obj
- link link3: geometry visual mesh filename=../../Model/meshes/visual/link3.obj
- link link4: geometry collision mesh filename=../../Model/meshes/collision/link4.obj; visual mesh filename=../../Model/meshes/visual/link4.obj
- link link5: geometry visual mesh filename=../../Model/meshes/visual/link5.obj
- link link6: geometry visual mesh filename=../../Model/meshes/visual/link6.obj
- link link7: geometry visual mesh filename=../../Model/meshes/visual/hand.obj; visual mesh filename=../../Model/meshes/visual/link7.obj
- link rightfinger: geometry visual mesh filename=../../Model/meshes/visual/finger.obj
