Commit message: cleaned up code and added dual arm sim stuff from panda starter code

File: 02-dual_arm_sim/dual_arm_mobile.urdf (robot description, URDF)
Before this commit: robot panda, 8 links, 7 joints
Links:
- removed link link0
- removed link link1
- removed link link2
- removed link link3
- removed link link4
- removed link link5
- removed link link6
- removed link link7
- added link leftfingerR, mass 0.1; visual mesh filename=../../../Model/meshes/visual/finger.obj
- added link link0R, mass 4; visual mesh filename=../../../Model/meshes/visual/link0.obj
- added link link1R, mass 3; visual mesh filename=../../../Model/meshes/visual/link1.obj
- added link link2R, mass 3; visual mesh filename=../../../Model/meshes/visual/link2.obj
- added link link3R, mass 2; visual mesh filename=../../../Model/meshes/visual/link3.obj
- added link link4R, mass 2; collision mesh filename=../../../Model/meshes/collision/link4.obj; visual mesh filename=../../../Model/meshes/visual/link4.obj
- added link link5R, mass 2; visual mesh filename=../../../Model/meshes/visual/link5.obj
- added link link6R, mass 1.5; visual mesh filename=../../../Model/meshes/visual/link6.obj
- added link link7R, mass 1.8; visual mesh filename=../../../Model/meshes/visual/hand.obj; visual mesh filename=../../../Model/meshes/visual/link7.obj
- added link rightfingerR, mass 0.1; visual mesh filename=../../../Model/meshes/visual/finger.obj
Joints:
- removed joint joint1
- removed joint joint2
- removed joint joint3
- removed joint joint4
- removed joint joint5
- removed joint joint6
- removed joint joint7
- added joint finger_joint1R: type prismatic, parent link7R, child leftfingerR, origin xyz=0 0 0.1654 rpy=0 0 -0.78539816339, axis 0 1 0, limit lower=0.0 upper=0.04 effort=20 velocity=0.2
- added joint finger_joint2R: type prismatic, parent link7R, child rightfingerR, origin xyz=0 0 0.1654 rpy=0 0 -0.78539816339, axis 0 1 0, limit lower=0.0 upper=0.04 effort=20 velocity=0.2
- added joint joint1R: type revolute, parent link0R, child link1R, origin xyz=0 0 0.333 rpy=0 0 0, axis 0 0 1, limit lower=-2.8973 upper=2.8973 effort=87 velocity=2.1750
- added joint joint2R: type revolute, parent link1R, child link2R, origin xyz=0 0 0 rpy=-1.57079632679 0 0, axis 0 0 1, limit lower=-1.7628 upper=1.7628 effort=87 velocity=2.1750
- added joint joint3R: type revolute, parent link2R, child link3R, origin xyz=0 -0.316 0 rpy=1.57079632679 0 0, axis 0 0 1, limit lower=-2.8973 upper=2.8973 effort=87 velocity=2.1750
- added joint joint4R: type revolute, parent link3R, child link4R, origin xyz=0.0825 0 0 rpy=1.57079632679 0 0, axis 0 0 1, limit lower=-3.0718 upper=-0.0698 effort=87 velocity=2.1750
- added joint joint5R: type revolute, parent link4R, child link5R, origin xyz=-0.0825 0.384 0 rpy=-1.57079632679 0 0, axis 0 0 1, limit lower=-2.8973 upper=2.8973 effort=12 velocity=2.6100
- added joint joint6R: type revolute, parent link5R, child link6R, origin xyz=0 0 0 rpy=1.57079632679 0 0, axis 0 0 1, limit lower=-0.0175 upper=3.7525 effort=12 velocity=2.6100
- added joint joint7R: type revolute, parent link6R, child link7R, origin xyz=0.088 0 0 rpy=1.57079632679 0 0, axis 0 0 1, limit lower=-2.8973 upper=2.8973 effort=12 velocity=2.6100
