Commit message: removed print statements for pose

File: 02-dual_arm_sim/mobilebase.urdf (robot description, URDF)
Before this commit: robot mobilebase, 5 links, 4 joints
Links:
- added link leftfingerL, mass 0.1; visual mesh filename=../../../Model/meshes/visual/finger.obj
- added link leftfingerR, mass 0.1; visual mesh filename=../../../Model/meshes/visual/finger.obj
- added link link0L, mass 4; visual mesh filename=../../../Model/meshes/visual/link0.obj
- added link link0R, mass 4; visual mesh filename=../../../Model/meshes/visual/link0.obj
- added link link1L, mass 3; visual mesh filename=../../../Model/meshes/visual/link1.obj
- added link link1R, mass 3; visual mesh filename=../../../Model/meshes/visual/link1.obj
- added link link2L, mass 3; visual mesh filename=../../../Model/meshes/visual/link2.obj
- added link link2R, mass 3; visual mesh filename=../../../Model/meshes/visual/link2.obj
- added link link3L, mass 2; visual mesh filename=../../../Model/meshes/visual/link3.obj
- added link link3R, mass 2; visual mesh filename=../../../Model/meshes/visual/link3.obj
- added link link4L, mass 2; collision mesh filename=../../../Model/meshes/collision/link4.obj; visual mesh filename=../../../Model/meshes/visual/link4.obj
- added link link4R, mass 2; collision mesh filename=../../../Model/meshes/collision/link4.obj; visual mesh filename=../../../Model/meshes/visual/link4.obj
- added link link5L, mass 2; visual mesh filename=../../../Model/meshes/visual/link5.obj
- added link link5R, mass 2; visual mesh filename=../../../Model/meshes/visual/link5.obj
- added link link6L, mass 1.5; visual mesh filename=../../../Model/meshes/visual/link6.obj
- added link link6R, mass 1.5; visual mesh filename=../../../Model/meshes/visual/link6.obj
- added link link7L, mass 1.8; visual mesh filename=../../../Model/meshes/visual/hand.obj; visual mesh filename=../../../Model/meshes/visual/link7.obj
- added link link7R, mass 1.8; visual mesh filename=../../../Model/meshes/visual/hand.obj; visual mesh filename=../../../Model/meshes/visual/link7.obj
- added link rightfingerL, mass 0.1; visual mesh filename=../../../Model/meshes/visual/finger.obj
- added link rightfingerR, mass 0.1; visual mesh filename=../../../Model/meshes/visual/finger.obj
- link base_link: mass 36.127263320367 -> 38.152
- link torso: mass 8.50250811972898 -> 8.5025
Joints:
- added joint finger_joint1L: type prismatic, parent link7L, child leftfingerL, origin xyz=0 0 0.1654 rpy=0 0 -0.78539816339, axis 0 1 0, limit lower=0.0 upper=0.04 effort=20 velocity=0.2
- added joint finger_joint1R: type prismatic, parent link7R, child leftfingerR, origin xyz=0 0 0.1654 rpy=0 0 -0.78539816339, axis 0 1 0, limit lower=0.0 upper=0.04 effort=20 velocity=0.2
- added joint finger_joint2L: type prismatic, parent link7L, child rightfingerL, origin xyz=0 0 0.1654 rpy=0 0 -0.78539816339, axis 0 1 0, limit lower=0.0 upper=0.04 effort=20 velocity=0.2
- added joint finger_joint2R: type prismatic, parent link7R, child rightfingerR, origin xyz=0 0 0.1654 rpy=0 0 -0.78539816339, axis 0 1 0, limit lower=0.0 upper=0.04 effort=20 velocity=0.2
- added joint joint1L: type revolute, parent link0L, child link1L, origin xyz=0 0 0.333 rpy=0 0 0, axis 0 0 1, limit lower=-2.8973 upper=2.8973 effort=87 velocity=2.1750
- added joint joint1R: type revolute, parent link0R, child link1R, origin xyz=0 0 0.333 rpy=0 0 0, axis 0 0 1, limit lower=-2.8973 upper=2.8973 effort=87 velocity=2.1750
- added joint joint2L: type revolute, parent link1L, child link2L, origin xyz=0 0 0 rpy=-1.57079632679 0 0, axis 0 0 1, limit lower=-1.7628 upper=1.7628 effort=87 velocity=2.1750
- added joint joint2R: type revolute, parent link1R, child link2R, origin xyz=0 0 0 rpy=-1.57079632679 0 0, axis 0 0 1, limit lower=-1.7628 upper=1.7628 effort=87 velocity=2.1750
- added joint joint3L: type revolute, parent link2L, child link3L, origin xyz=0 -0.316 0 rpy=1.57079632679 0 0, axis 0 0 1, limit lower=-2.8973 upper=2.8973 effort=87 velocity=2.1750
- added joint joint3R: type revolute, parent link2R, child link3R, origin xyz=0 -0.316 0 rpy=1.57079632679 0 0, axis 0 0 1, limit lower=-2.8973 upper=2.8973 effort=87 velocity=2.1750
- added joint joint4L: type revolute, parent link3L, child link4L, origin xyz=0.0825 0 0 rpy=1.57079632679 0 0, axis 0 0 1, limit lower=-3.0718 upper=-0.0698 effort=87 velocity=2.1750
- added joint joint4R: type revolute, parent link3R, child link4R, origin xyz=0.0825 0 0 rpy=1.57079632679 0 0, axis 0 0 1, limit lower=-3.0718 upper=-0.0698 effort=87 velocity=2.1750
- added joint joint5L: type revolute, parent link4L, child link5L, origin xyz=-0.0825 0.384 0 rpy=-1.57079632679 0 0, axis 0 0 1, limit lower=-2.8973 upper=2.8973 effort=12 velocity=2.6100
- added joint joint5R: type revolute, parent link4R, child link5R, origin xyz=-0.0825 0.384 0 rpy=-1.57079632679 0 0, axis 0 0 1, limit lower=-2.8973 upper=2.8973 effort=12 velocity=2.6100
- added joint joint6L: type revolute, parent link5L, child link6L, origin xyz=0 0 0 rpy=1.57079632679 0 0, axis 0 0 1, limit lower=-0.0175 upper=3.7525 effort=12 velocity=2.6100
- added joint joint6R: type revolute, parent link5R, child link6R, origin xyz=0 0 0 rpy=1.57079632679 0 0, axis 0 0 1, limit lower=-0.0175 upper=3.7525 effort=12 velocity=2.6100
- added joint joint7L: type revolute, parent link6L, child link7L, origin xyz=0.088 0 0 rpy=1.57079632679 0 0, axis 0 0 1, limit lower=-2.8973 upper=2.8973 effort=12 velocity=2.6100
- added joint joint7R: type revolute, parent link6R, child link7R, origin xyz=0.088 0 0 rpy=1.57079632679 0 0, axis 0 0 1, limit lower=-2.8973 upper=2.8973 effort=12 velocity=2.6100
- added joint torso to leftarm: type revolute, parent torso, child link0L, origin xyz=0 0.0 0.1 rpy=-1 0 0, axis 0 0 1, limit lower=0 upper=0 effort=0 velocity=0
- added joint torso to rightarm: type revolute, parent torso, child link0R, origin xyz=0 0.0 0.1 rpy=1 0 0, axis 0 0 1, limit lower=0 upper=0 effort=0 velocity=0
- joint prismatic: axis 0 1 0 -> 0 0 1; origin xyz=0.20408 -0.7946 0.4254 rpy=1.5708 0 0 -> xyz=0 0 0 rpy=0 0 0
